File: Schematics/DIHi Cheers.kicad_sch (KiCad schematic)
At the start: 12 parts, among them U1 SN74LVC1T45DBV, U10 SN74LVC1T45DBV, U11 SN74LVC1T45DBV, U2 SN74LVC1T45DBV, U3 SN74LVC1T45DBV, U4 SN74LVC1T45DBV, U5 SN74LVC1T45DBV, U6 SN74LVC1T45DBV, U7 SN74LVC1T45DBV, U8 SN74LVC1T45DBV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

Commit message: fixed shifting direction and added barrel jack for 5v power
Parts:
- added J1: Barrel_Jack, Connector_BarrelJack:BarrelJack_SwitchcraftConxall_RAPC10U_Horizontal, symbol Connector:Barrel_Jack
Connections:
- net +3.3V: now also U1.6 (VCCB), U10.6 (VCCB), U11.6 (VCCB), U2.6 (VCCB), U3.6 (VCCB), U4.6 (VCCB), U5.6 (VCCB), U6.6 (VCCB), U7.6 (VCCB), U8.6 (VCCB), U9.6 (VCCB), J1.2; no longer U1.1 (VCCA), U10.1 (VCCA), U11.1 (VCCA), U2.1 (VCCA), U3.1 (VCCA), U4.1 (VCCA), U5.1 (VCCA), U6.1 (VCCA), U7.1 (VCCA), U8.1 (VCCA), U9.1 (VCCA)
- net +5V: now also U1.1 (VCCA), U10.1 (VCCA), U11.1 (VCCA), U2.1 (VCCA), U3.1 (VCCA), U4.1 (VCCA), U5.1 (VCCA), U6.1 (VCCA), U7.1 (VCCA), U8.1 (VCCA), U9.1 (VCCA), J1.1; no longer U1.6 (VCCB), U10.6 (VCCB), U11.6 (VCCB), U2.6 (VCCB), U3.6 (VCCB), U4.6 (VCCB), U5.6 (VCCB), U6.6 (VCCB), U7.6 (VCCB), U8.6 (VCCB), U9.6 (VCCB)
